Commit message: Latest working changes

File: src/articubot_one/description/lidar.xacro (robot description, xacro)
@@ -4,5 +4,5 @@
         <parent link="chassis"/>
         <child link="laser_frame"/>
-        <origin xyz="0.122 0 0.112" rpy="0 0 0"/>
+        <origin xyz="0.122 0 0.112" rpy="0 0 3.14159"/>
     </joint>
     <link name="laser_frame">

File: src/articubot_one/description/robot_core.xacro (robot description, xacro)
@@ -2,14 +2,14 @@
 <robot xmlns:xacro="http://www.ros.org/wiki/xacro" >
     <xacro:include filename="inertial_macros.xacro"/>
-    <xacro:property name="chassis_length" value="0.2159"/>
+    <xacro:property name="chassis_length" value="0.22"/>
     <xacro:property name="chassis_width" value="0.1524"/>
     <xacro:property name="chassis_height" value="0.08255"/>
     <xacro:property name="chassis_mass" value="1.0"/>
-    <xacro:property name="wheel_radius" value="0.0381"/>
+    <xacro:property name="wheel_radius" value="0.04"/>
     <xacro:property name="wheel_thickness" value="0.01"/>
     <xacro:property name="wheel_mass" value="0.05"/>
-    <xacro:property name="wheel_offset_x" value="0.0254"/>
-    <xacro:property name="wheel_offset_y" value="0.1016"/>
-    <xacro:property name="wheel_offset_z" value="0.01"/>
+    <xacro:property name="wheel_offset_x" value="0.065"/>
+    <xacro:property name="wheel_offset_y" value="0.1038"/>
+    <xacro:property name="wheel_offset_z" value="0.02"/>
     <xacro:property name="caster_wheel_radius" value="0.015"/>
     <xacro:property name="caster_wheel_mass" value="0.01"/>
@@ -54,5 +54,5 @@
                 <box size="${chassis_length} ${chassis_width} ${chassis_height}"/>
             </geometry>
-            <material name="orange"/>
+            <material name="white"/>
         </visual>
         <collision>
@@ -81,5 +81,5 @@
                 <cylinder radius="${wheel_radius}" length="${wheel_thickness}"/>
             </geometry>
-            <material name="blue"/>
+            <material name="black"/>
         </visual>
         <collision>
@@ -107,5 +107,5 @@
                 <cylinder radius="${wheel_radius}" length="${wheel_thickness}"/>
             </geometry>
-            <material name="blue"/>
+            <material name="black"/>
         </visual>
         <collision>

File: src/articubot_one/description/ros2_control.xacro (robot description, xacro)
@@ -15,6 +15,6 @@
             <joint name="left_wheel_joint">
                 <command_interface name="velocity">
-                    <param name="min">-10</param>
-                    <param name="max">10</param>
+                    <param name="min">-1</param>
+                    <param name="max">1</param>
                 </command_interface>
                 <state_interface name="position"/>
@@ -23,6 +23,6 @@
             <joint name="right_wheel_joint">
                 <command_interface name="velocity">
-                    <param name="min">-10</param>
-                    <param name="max">10</param>
+                    <param name="min">-1</param>
+                    <param name="max">1</param>
                 </command_interface>
                 <state_interface name="position"/>
@@ -38,6 +38,6 @@
             <joint name="left_wheel_joint">
                 <command_interface name="velocity">
-                    <param name="min">-10</param>
-                    <param name="max">10</param>
+                    <param name="min">-1</param>
+                    <param name="max">1</param>
                 </command_interface>
                 <state_interface name="velocity"/>
@@ -46,6 +46,6 @@
             <joint name="right_wheel_joint">
                 <command_interface name="velocity">
-                    <param name="min">-10</param>
-                    <param name="max">10</param>
+                    <param name="min">-1</param>
+                    <param name="max">1</param>
                 </command_interface>
                 <state_interface name="velocity"/>
