Commit message: Adds camera URDF

File: src/articubot_one/description/camera.xacro (robot description, xacro)
@@ -4,17 +4,17 @@
         <parent link="chassis"/>
         <child link="camera_link"/>
-        <origin xyz="0.276 0 0.181" rpy="0 0.18 0"/>
+        <origin xyz="0.26 0.00 0.07" rpy="0 0 0"/>
     </joint>
     <link name="camera_link">
         <visual>
             <geometry>
-                <box size="0.010 0.03 0.03"/>
+                <box size="0.01 0.08 0.03"/>
             </geometry>
-            <material name="black"/>
+            <material name="black"/>0.09
         </visual>
         <visual>
-            <origin xyz="0 0 -0.05"/>
+            <origin xyz="-0.04 0 0.01" rpy="0 ${-pi/2} 0"/>
             <geometry>
-                <cylinder radius="0.002" length="0.1"/>
+                <cylinder radius="0.002" length="0.08"/>
             </geometry>
             <material name="black"/>

Commit message: Attempting to add range layer to nav2

File: src/articubot_one/description/camera.xacro (robot description, xacro)
@@ -7,4 +7,9 @@
     </joint>
     <link name="camera_link">
+        <collision>
+            <geometry>
+                <box size="0.05 0.1 0.09"/>
+            </geometry>
+        </collision>
         <visual>
             <geometry>

File: src/articubot_one/description/ultrasonic_sensor.xacro (robot description, xacro)
@@ -32,6 +32,6 @@
                 <samples>5</samples>
                 <resolution>1.000000</resolution>
-                <min_angle>-0.12</min_angle>
-                <max_angle>0.12</max_angle>
+                <min_angle>-0.3</min_angle>
+                <max_angle>0.3</max_angle>
                 </horizontal>
                 <vertical>
@@ -44,5 +44,5 @@
             <range>
                 <min>0.05</min>
-                <max>12</max>
+                <max>40</max>
                 <resolution>0.01</resolution>
             </range>
@@ -53,11 +53,11 @@
             </noise>
             </ray>
-            <plugin name="ultrasonic_sensor_1" filename="libgazebo_ros_ray_sensor.so">
+            <plugin name="ultrasonic_sensor" filename="libgazebo_ros_ray_sensor.so">
             <ros>
-                <remapping>~/out:=ultrasonic_sensor_1</remapping>
+                <remapping>~/out:=ultrasonic_sensor</remapping>
             </ros>
             <output_type>sensor_msgs/Range</output_type>
             <radiation_type>ultrasound</radiation_type>
-            <frame_name>ultrasonic_1_link</frame_name>
+            <frame_name>ultrasonic_link</frame_name>
             </plugin>
         </sensor>
